File: Hardware/SparkFun_Ublox SAM-M8Q.brd (EAGLE design)
At the start: 40.6 x 40.6 mm, 75 parts, among them J1 Qwiic Right Angle, J2 Qwiic Right Angle, J4 BOOT, U1 UBLOX_SAM_M8Q-0-10

Commit message: Adds measurments to measures layer, fixes power LED air wire, adjusts bottom dimension line
Other:
- board text added: "+"
- board text added: "-"
Changed lines of the file:
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@@
 <layer number="115" name="ReferenceISLANDS" color="7" fill="1" visible="no" active="no"/>
 <layer number="116" name="Patch_BOT" color="9" fill="4" visible="no" active="no"/>
-<layer number="117" name="PM_Ref" color="26" fill="1" visible="yes" active="yes"/>
+<layer number="117" name="PM_Ref" color="26" fill="1" visible="no" active="yes"/>
 <layer number="118" name="Rect_Pads" color="7" fill="1" visible="no" active="no"/>
-<layer number="119" name="PF_Ref" color="31" fill="1" visible="yes" active="yes"/>
-<layer number="120" name="WFL_Ref" color="25" fill="1" visible="yes" active="yes"/>
+<layer number="119" name="PF_Ref" color="31" fill="1" visible="no" active="yes"/>
+<layer number="120" name="WFL_Ref" color="25" fill="1" visible="no" active="yes"/>
 <layer number="121" name="_tsilk" color="7" fill="1" visible="no" active="no"/>
 <layer number="122" name="_bsilk" color="7" fill="1" visible="no" active="no"/>
@@
 <wire x1="0" y1="40.64" x2="40.64" y2="40.64" width="0.2032" layer="20"/>
 <wire x1="40.64" y1="40.64" x2="40.64" y2="0" width="0.2032" layer="20"/>
-<wire x1="40.64" y1="0" x2="0" y2="0" width="0.1524" layer="20"/>
+<wire x1="40.64" y1="0" x2="0" y2="0" width="0.2032" layer="20"/>
 <text x="34.417" y="1.27" size="1.27" layer="16" font="vector" ratio="15" rot="MR180" align="center">v10</text>
-<text x="-2.54" y="-8.89" size="1.778" layer="47">Measurements in inches</text>
+<text x="3.302" y="49.022" size="1.778" layer="47" font="vector">Measurements in inches</text>
 <wire x1="12.7" y1="40.64" x2="12.7" y2="38.1" width="0.1778" layer="21"/>
 <wire x1="27.94" y1="38.1" x2="27.94" y2="40.64" width="0.1778" layer="21"/>
@@
 <text x="12.7" y="-17.78" size="1.778" layer="51" font="vector">Nathan Seidle</text>
 <text x="-6.35" y="-20.574" size="1.778" layer="51" font="vector">Revised By: Elias Santistevan</text>
+<text x="0.508" y="29.21" size="1.27" layer="21" font="vector" ratio="15">+</text>
+<text x="0.508" y="32.766" size="1.27" layer="21" font="vector" ratio="15">-</text>
+<dimension x1="0" y1="40.64" x2="40.64" y2="40.64" x3="20.32" y3="44.45" textsize="1.27" textratio="15" layer="47" unit="inch"/>
+<dimension x1="40.64" y1="40.64" x2="40.64" y2="0" x3="47.752" y3="20.32" textsize="1.27" textratio="15" layer="47" unit="inch"/>
 </plain>
 <attributes>
@@
 <wire x1="13.195" y1="22.22" x2="9.52" y2="22.22" width="0.3048" layer="1"/>
 <wire x1="9.52" y1="22.22" x2="8.12" y2="20.82" width="0.3048" layer="1"/>
-<wire x1="31.877" y1="2.667" x2="24.13" y2="2.667" width="0.3048" layer="16"/>
+<wire x1="32.0548" y1="2.667" x2="24.13" y2="2.667" width="0.3048" layer="16"/>
 <wire x1="24.13" y1="2.667" x2="7.493" y2="2.667" width="0.3048" layer="16"/>
 <wire x1="7.493" y1="2.667" x2="1.27" y2="8.89" width="0.3048" layer="16"/>
 <wire x1="1.27" y1="8.89" x2="1.27" y2="20.32" width="0.3048" layer="16"/>
 <via x="1.27" y="20.32" extent="1-16" drill="0.381"/>
-<wire x1="31.877" y1="2.667" x2="35.56" y2="6.35" width="0.3048" layer="16"/>
-<wire x1="35.56" y1="6.35" x2="39.37" y2="10.16" width="0.3048" layer="16"/>
-<wire x1="39.37" y1="10.16" x2="39.37" y2="19.05" width="0.3048" layer="16"/>
+<wire x1="32.0548" y1="2.667" x2="35.56" y2="6.1722" width="0.3048" layer="16"/>
+<wire x1="35.56" y1="6.1722" x2="39.37" y2="9.9822" width="0.3048" layer="16"/>
+<wire x1="39.37" y1="9.9822" x2="39.37" y2="19.05" width="0.3048" layer="16"/>
 <wire x1="39.37" y1="19.05" x2="39.37" y2="30.48" width="0.3048" layer="16"/>
 <wire x1="39.37" y1="19.05" x2="38.6" y2="19.82" width="0.3048" layer="1"/>
@@
 <wire x1="3.39" y1="18.2" x2="2.54" y2="19.05" width="0.3048" layer="1"/>
 <wire x1="2.54" y1="19.05" x2="2.54" y2="20.82" width="0.3048" layer="1"/>
-<via x="35.56" y="6.35" extent="1-16" drill="0.381"/>
+<via x="35.56" y="6.1722" extent="1-16" drill="0.381"/>
 <contactref element="JP2" pad="2"/>
 <wire x1="38.6" y1="19.82" x2="37.846" y2="19.82" width="0.3048" layer="1"/>
@@
 <wire x1="36.195" y1="15.875" x2="37.846" y2="17.526" width="0.254" layer="1"/>
 <wire x1="37.846" y1="17.526" x2="37.846" y2="19.82" width="0.254" layer="1"/>
-<wire x1="35.56" y1="6.35" x2="35.56" y2="7.62" width="0.254" layer="1"/>
+<wire x1="35.56" y1="6.1722" x2="35.56" y2="7.62" width="0.254" layer="1"/>
 <contactref element="J3" pad="3"/>
 <wire x1="24.13" y1="1.27" x2="24.13" y2="2.667" width="0.3048" layer="16"/>
@@
 <via x="19.812" y="7.874" extent="1-16" drill="0.381"/>
 <via x="7.874" y="23.114" extent="1-16" drill="0.381"/>
-<wire x1="37.35" y1="26.543" x2="33.02" y2="24.13" width="0" layer="19" extent="1-1"/>
+<via x="35.814" y="25.654" extent="1-16" drill="0.381"/>
 </signal>
 <signal name="SCL">
